Commit message: refactor: initial refactor of Pro630 Gazebo project

File: mycobot_pro/mycobotpro630_gazeboros2/config/firefighter.ros2_control.xacro (robot description, xacro)
@@ -2,7 +2,8 @@
 <robot xmlns:xacro="http://www.ros.org/wiki/xacro">
     <xacro:macro name="firefighter_ros2_control" params="name initial_positions_file">
-        <xacro:property name="initial_positions" value="${load_yaml(initial_positions_file)['initial_positions']}"/>
+        <xacro:property name="initial_positions" value="${xacro.load_yaml(initial_positions_file)['initial_positions']}"/>
         <ros2_control name="${name}" type="system">
             <hardware>
+                <!-- By default, set up controllers for simulation. This won't work on real hardware -->
                 <plugin>gazebo_ros2_control/GazeboSystem</plugin>
             </hardware>
@@ -56,4 +57,52 @@
                 <state_interface name="velocity"/>
             </joint>
+            <!-- Keep all gripper joints in the same GazeboSystem update.
+                 The separate mimic plugins set fmax to the effort limit and
+                 changed positions without resetting their residual velocity. -->
+            <joint name="gripper_base_to_gripper_left2">
+                <param name="mimic">gripper_controller</param>
+                <param name="multiplier">1.0</param>
+                <command_interface name="position"/>
+                <state_interface name="position">
+                  <param name="initial_value">${initial_positions['gripper_controller']}</param>
+                </state_interface>
+                <state_interface name="velocity"/>
+            </joint>
+            <joint name="gripper_left3_to_gripper_left1">
+                <param name="mimic">gripper_controller</param>
+                <param name="multiplier">-1.0</param>
+                <command_interface name="position"/>
+                <state_interface name="position">
+                  <param name="initial_value">${-initial_positions['gripper_controller']}</param>
+                </state_interface>
+                <state_interface name="velocity"/>
+            </joint>
+            <joint name="gripper_base_to_gripper_right3">
+                <param name="mimic">gripper_controller</param>
+                <param name="multiplier">-1.0</param>
+                <command_interface name="position"/>
+                <state_interface name="position">
+                  <param name="initial_value">${-initial_positions['gripper_controller']}</param>
+                </state_interface>
+                <state_interface name="velocity"/>
+            </joint>
+            <joint name="gripper_base_to_gripper_right2">
+                <param name="mimic">gripper_controller</param>
+                <param name="multiplier">-1.0</param>
+                <command_interface name="position"/>
+                <state_interface name="position">
+                  <param name="initial_value">${-initial_positions['gripper_controller']}</param>
+                </state_interface>
+                <state_interface name="velocity"/>
+            </joint>
+            <joint name="gripper_right3_to_gripper_right1">
+                <param name="mimic">gripper_controller</param>
+                <param name="multiplier">1.0</param>
+                <command_interface name="position"/>
+                <state_interface name="position">
+                  <param name="initial_value">${initial_positions['gripper_controller']}</param>
+                </state_interface>
+                <state_interface name="velocity"/>
+            </joint>
         </ros2_control>
     </xacro:macro>

File: mycobot_pro/mycobotpro630_gazeboros2/config/firefighter.urdf.xacro (robot description, xacro)
@@ -2,4 +2,8 @@
 <robot xmlns:xacro="http://www.ros.org/wiki/xacro" name="firefighter">
     <xacro:arg name="initial_positions_file" default="initial_positions.yaml" />
+    <!-- MoveIt uses collision_exact by default. Gazebo overrides this with
+         collision_gazebo because ODE is unstable with dynamic non-convex,
+         high-triangle collision meshes. -->
+    <xacro:arg name="collision_mesh_dir" default="collision_exact" />
     <!-- Import firefighter urdf file -->
     <xacro:include filename="$(find mycobotpro630_gazeboros2)/config/mycobot_pro_630_force_gripper.urdf" />
@@ -7,3 +11,15 @@
     <xacro:include filename="firefighter.ros2_control.xacro" />
     <xacro:firefighter_ros2_control name="FakeSystem" initial_positions_file="$(arg initial_positions_file)"/>
+    <gazebo>
+        <plugin filename="libgazebo_ros2_control.so" name="gazebo_ros2_control">
+            <parameters>$(find mycobotpro630_gazeboros2)/config/ros2_controllers.yaml</parameters>
+            <!-- The Gazebo entity is spawned from the namespaced description
+                 publisher because it uses collision_gazebo and, in real-pose
+                 mirror mode, the read-only hardware snapshot.  Do not let the
+                 plugin fall back to the MoveIt robot_state_publisher, whose
+                 ros2_control initial values are the default zero pose. -->
+            <robot_param>robot_description</robot_param>
+            <robot_param_node>/gazebo_spawn/robot_description_publisher</robot_param_node>
+        </plugin>
+    </gazebo>
 </robot>

File: mycobot_pro/mycobotpro630_gazeboros2/config/mycobot_pro_630_force_gripper.urdf (robot description, URDF)
Before this commit: robot firefighter, 16 links, 15 joints
Links:
- added link gripper_cable_terminal, mass 0.000001; collision cylinder length=0.025 radius=0.006624266
- link base: geometry collision mesh filename=package://mycobot_description/urdf/mycobot_pro_630/$(arg co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; visual mesh filename=package://mycobot_description/urdf/mycobot_pro_630/base.dae
- link gripper_base: mass 0.005 -> 0.12; geometry collision mesh filename=package://mycobot_description/urdf/mycobot_pro_630/$(arg co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; visual mesh filename=package://mycobot_description/urdf/mycobot_320_m5_2022/forc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
- link gripper_connection: mass 0.1 -> 0.15; geometry collision mesh filename=package://mycobot_description/urdf/mycobot_pro_630/$(arg co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; visual mesh filename=package://mycobot_description/urdf/mycobot_320_m5_2022/forc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
- link gripper_left1: mass 0.005 -> 0.02; geometry collision mesh filename=package://mycobot_description/urdf/mycobot_pro_630/$(arg co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; visual mesh filename=package://mycobot_description/urdf/mycobot_320_m5_2022/forc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
- link gripper_left2: mass 0.005 -> 0.02; geometry collision mesh filename=package://mycobot_description/urdf/mycobot_pro_630/$(arg co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; visual mesh filename=package://mycobot_description/urdf/mycobot_320_m5_2022/forc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
- link gripper_left3: mass 0.005 -> 0.02; geometry collision mesh filename=package://mycobot_description/urdf/mycobot_pro_630/$(arg co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; visual mesh filename=package://mycobot_description/urdf/mycobot_320_m5_2022/forc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
- link gripper_right1: mass 0.005 -> 0.02; geometry collision mesh filename=package://mycobot_description/urdf/mycobot_pro_630/$(arg co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; visual mesh filename=package://mycobot_description/urdf/mycobot_320_m5_2022/forc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
- link gripper_right2: mass 0.005 -> 0.02; geometry collision mesh filename=package://mycobot_description/urdf/mycobot_pro_630/$(arg co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; visual mesh filename=package://mycobot_description/urdf/mycobot_320_m5_2022/forc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
- link gripper_right3: mass 0.005 -> 0.02; geometry collision mesh filename=package://mycobot_description/urdf/mycobot_pro_630/$(arg co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; visual mesh filename=package://mycobot_description/urdf/mycobot_320_m5_2022/forc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
- link link1: geometry collision mesh filename=package://mycobot_description/urdf/mycobot_pro_630/$(arg co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; visual mesh filename=package://mycobot_description/urdf/mycobot_pro_630/link1.dae
- link link2: geometry collision mesh filename=package://mycobot_description/urdf/mycobot_pro_630/$(arg co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; visual mesh filename=package://mycobot_description/urdf/mycobot_pro_630/link2.dae
- link link3: geometry collision mesh filename=package://mycobot_description/urdf/mycobot_pro_630/$(arg co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; visual mesh filename=package://mycobot_description/urdf/mycobot_pro_630/link3.dae
- link link4: geometry collision mesh filename=package://mycobot_description/urdf/mycobot_pro_630/$(arg co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; visual mesh filename=package://mycobot_description/urdf/mycobot_pro_630/link4.dae
- link link5: geometry collision mesh filename=package://mycobot_description/urdf/mycobot_pro_630/$(arg co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; visual mesh filename=package://mycobot_description/urdf/mycobot_pro_630/link5.dae
- link link6: geometry collision mesh filename=package://mycobot_description/urdf/mycobot_pro_630/$(arg co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; visual mesh filename=package://mycobot_description/urdf/mycobot_pro_630/link6.dae
Joints:
- added joint gripper_base_to_cable_terminal: type fixed, parent gripper_base, child gripper_cable_terminal, origin xyz=-0.107 0.012 0.0 rpy=1.5708 0 1.5708

Commit message: feat: add support for grippers with and without force control

File: mycobot_pro/mycobotpro630_gazeboros2/config/firefighter.ros2_control.xacro (robot description, xacro)
@@ -50,4 +50,5 @@
                 <state_interface name="velocity"/>
             </joint>
+            <xacro:if value="$(arg with_gripper)">
             <joint name="gripper_controller">
                 <command_interface name="position"/>
@@ -105,4 +106,5 @@
                 <state_interface name="velocity"/>
             </joint>
+            </xacro:if>
         </ros2_control>
     </xacro:macro>

File: mycobot_pro/mycobotpro630_gazeboros2/config/firefighter.urdf.xacro (robot description, xacro)
@@ -1,4 +1,8 @@
 <?xml version="1.0"?>
 <robot xmlns:xacro="http://www.ros.org/wiki/xacro" name="firefighter">
+    <xacro:arg name="with_gripper" default="true" />
+    <!-- Internal mirror setting; simulation and MoveIt retain normal collisions. -->
+    <xacro:arg name="gazebo_contact_response" default="true" />
+    <xacro:arg name="controller_config_file" default="$(find mycobotpro630_gazeboros2)/config/ros2_controllers.yaml" />
     <xacro:arg name="initial_positions_file" default="initial_positions.yaml" />
     <!-- MoveIt uses collision_exact by default. Gazebo overrides this with
@@ -13,5 +17,5 @@
     <gazebo>
         <plugin filename="libgazebo_ros2_control.so" name="gazebo_ros2_control">
-            <parameters>$(find mycobotpro630_gazeboros2)/config/ros2_controllers.yaml</parameters>
+            <parameters>$(arg controller_config_file)</parameters>
             <!-- The Gazebo entity is spawned from the namespaced description
                  publisher because it uses collision_gazebo and, in real-pose

File: mycobot_pro/mycobotpro630_gazeboros2/config/mycobot_pro_630_force_gripper.urdf (robot description, URDF)
Before this commit: robot firefighter, 17 links, 16 joints
Links:
- removed link gripper_base
- removed link gripper_cable_terminal
- removed link gripper_connection
- removed link gripper_left1
- removed link gripper_left2
- removed link gripper_left3
- removed link gripper_right1
- removed link gripper_right2
- removed link gripper_right3
Joints:
- removed joint gripper_base_to_cable_terminal
- removed joint gripper_base_to_gripper_left2
- removed joint gripper_base_to_gripper_right2
- removed joint gripper_base_to_gripper_right3
- removed joint gripper_controller
- removed joint gripper_left3_to_gripper_left1
- removed joint gripper_right3_to_gripper_right1
- removed joint joint6_to_gripper_base
- removed joint joint6_to_gripper_connect
